Commit message: 完善了启动文件，把多余的ros2_control_node启动删掉，解决了启动时无用的报错信息；增加了rviz2启动，解决了urdf中轮子关节state_interface没有加position导致rviz2启动 时transform报错的问题

File: ros2_ws/src/ustb_doggo_urdf/urdf/ustb_doggo_urdf.urdf (robot description, URDF)
Before this commit: robot ustb_doggo_urdf, 21 links, 20 joints
Links:
- added link laser_link, mass 0.0001; collision box size=0.01 0.01 0.01; visual box size=0.1 0.1 0.1
Joints:
- added joint joint_laser: type fixed, parent base_link, child laser_link, origin xyz=0 0 0.09 rpy=0 0 -1.57079633, axis 0 0 -1

Commit message: 增加建图功能，需要apt安装slam-toolbox

File: ros2_ws/src/ustb_doggo_urdf/urdf/ustb_doggo_urdf.urdf (robot description, URDF)
Before this commit: robot ustb_doggo_urdf, 22 links, 21 joints
Links:
- link laser_link: geometry collision box size=0.001 0.001 0.001; visual box size=0.1 0.1 0.1
Joints:
- joint joint_laser: origin xyz=0 0 0.09 rpy=0 0 -1.57079633 -> xyz=0 0 0.1 rpy=0 0 -1.57079633

Commit message: 增加激光雷达里程计rf2o和imu，通过robot_localization的ekf节点进行融合；解决了ekf在只有rf2o输入时不发布tf的问题，原因是ekf配置odom+id需要id按顺序配置，即先有odom0才能有odom1

File: ros2_ws/src/ustb_doggo_urdf/urdf/ustb_doggo_urdf.urdf (robot description, URDF)
Before this commit: robot ustb_doggo_urdf, 22 links, 21 joints
Links:
- added link imu_link, mass 0.001; collision box size=0.001 0.001 0.001; visual box size=0.001 0.001 0.001
Joints:
- added joint imu_joint: type fixed, parent base_link, child imu_link, origin xyz=0.0235 0 0.0351 rpy=0 0 0, axis 0 0 0
- joint joint_laser: origin xyz=0 0 0.1 rpy=0 0 -1.57079633 -> xyz=0 0 0.1 rpy=0 0 0
